Commit message: Update urdf with working mesh locations

File: Nav2Stuff/robocad/tum/robot.urdf (robot description, URDF)
Before this commit: robot Tum_onshape, 5 links, 4 joints
Links:
- link base_link: geometry collision mesh filename=file:///TumDWM1001/Nav2Stuff/robocad/tum/base_link.stl; visual mesh filename=file:///TumDWM1001/Nav2Stuff/robocad/tum/base_link.stl
- link part_1: geometry collision mesh filename=file:///TumDWM1001/Nav2Stuff/robocad/tum/part_1.stl; visual mesh filename=file:///TumDWM1001/Nav2Stuff/robocad/tum/part_1.stl
- link part_1_2: geometry collision mesh filename=file:///TumDWM1001/Nav2Stuff/robocad/tum/part_1.stl; visual mesh filename=file:///TumDWM1001/Nav2Stuff/robocad/tum/part_1.stl
- link part_1_3: geometry collision mesh filename=file:///TumDWM1001/Nav2Stuff/robocad/tum/part_1.stl; visual mesh filename=file:///TumDWM1001/Nav2Stuff/robocad/tum/part_1.stl
- link part_1_4: geometry collision mesh filename=file:///TumDWM1001/Nav2Stuff/robocad/tum/part_1.stl; visual mesh filename=file:///TumDWM1001/Nav2Stuff/robocad/tum/part_1.stl

Commit message: test URDF

File: Nav2Stuff/robocad/tum/robot.urdf (robot description, URDF)
Before this commit: robot sam_bot, 5 links, 4 joints
Joints:
- joint wheel1_speed: type revolute -> continuous
