Commit message: Update robot.urdf

File: Nav2Stuff/robocad/tum2/robot.urdf (robot description, URDF)
Before this commit: robot onshape, 10 links, 9 joints
Links:
- link base_link: geometry collision mesh filename=file:///TumDWM1001/Nav2Stuff/robocad/tum2/base_link.stl; visual mesh filename=file:///TumDWM1001/Nav2Stuff/robocad/tum2/base_link.stl
- link wheel_link: geometry collision mesh filename=file:///TumDWM1001/Nav2Stuff/robocad/tum2/wheel_link.stl; visual mesh filename=file:///TumDWM1001/Nav2Stuff/robocad/tum2/wheel_link.stl
- link wheel_link_2: geometry collision mesh filename=file:///TumDWM1001/Nav2Stuff/robocad/tum2/wheel_link.stl; visual mesh filename=file:///TumDWM1001/Nav2Stuff/robocad/tum2/wheel_link.stl
- link wheel_link_3: geometry collision mesh filename=file:///TumDWM1001/Nav2Stuff/robocad/tum2/wheel_link.stl; visual mesh filename=file:///TumDWM1001/Nav2Stuff/robocad/tum2/wheel_link.stl
- link wheel_link_4: geometry collision mesh filename=file:///TumDWM1001/Nav2Stuff/robocad/tum2/wheel_link.stl; visual mesh filename=file:///TumDWM1001/Nav2Stuff/robocad/tum2/wheel_link.stl

Commit message: retry URDF

File: Nav2Stuff/robocad/tum2/robot.urdf (robot description, URDF)
Before this commit: robot onshape, 10 links, 9 joints
Links:
- link base_link: mass 0.4998587895360000477 -> 0.49985878953600015873
Joints:
- joint base_frame: origin xyz=0 -5.5511151231257827021e-17 0.050799999999999997935 rpy=0 -0 0 -> xyz=-0.0063901649612328748074 -0.00027908066273285223047 0.052450807481831340784 rpy=0 -0 0
- joint wheel1: origin xyz=0.20320000000000010276 0.10159999999999996811 0.025400000000000005906 rpy=1.570796326794896558 -0 1.570796326794896558 -> xyz=0.19612022438614162834 0.098613027984792461789 0.027050807481831352225 rpy=1.570796326794896558 -0 1.570796326794896558
- joint wheel1_frame: origin xyz=0 0 0 rpy=3.141592653589793116 -0 1.570796326794896558 -> xyz=0.0027078913524746783814 0.012499999999999997224 0.01181038934737443924 rpy=1.570796326794896558 1.570796326794896558 0; parent wheel_link_3 -> wheel_link_4
- joint wheel2: origin xyz=0.20320000000000004725 -0.10160000000000005138 0.025400000000000005906 rpy=1.570796326794896558 -0 1.570796326794896558 -> xyz=0.19612022438614157283 -0.10458697201520755771 0.027050807481831348755 rpy=1.570796326794896558 -0 1.570796326794896558
- joint wheel2_frame: origin xyz=-1.3877787807814456755e-17 0 0 rpy=3.141592653589793116 -0 1.570796326794896558 -> xyz=0.0027078913524746922592 0.012499999999999997224 0.01181038934737443924 rpy=1.570796326794896558 1.570796326794896558 0; parent wheel_link_4 -> wheel_link_3
- joint wheel3: origin xyz=-0.20319999999999999174 0.10159999999999999587 0.025400000000000005906 rpy=-1.570796326794896558 -0 1.570796326794896558 -> xyz=-0.21027977561385843841 0.098613027984792489544 0.027050807481831348755 rpy=-1.570796326794896558 -0 1.570796326794896558
- joint wheel3_frame: origin xyz=0 0 0 rpy=3.141592653589793116 -0 1.570796326794896558 -> xyz=0.0027078913524746783814 -0.012500000000000000694 0.013189610652625555209 rpy=-1.570796326794896558 -1.570796326794896558 0
- joint wheel4: origin xyz=-0.20320000000000004725 -0.10160000000000000975 0.025400000000000005906 rpy=-1.570796326794896558 -0 1.570796326794896558 -> xyz=-0.21027977561385849392 -0.10458697201520752995 0.027050807481831348755 rpy=-1.570796326794896558 -0 1.570796326794896558
- joint wheel4_frame: origin xyz=2.7755575615628913511e-17 0 0 rpy=3.141592653589793116 -0 1.570796326794896558 -> xyz=0.0027078913524746922592 -0.012499999999999997224 0.013189610652625582965 rpy=-1.570796326794896558 -1.570796326794896558 0
