Commit message: Update robot.urdf

File: Nav2Stuff/robocad/tum_block/robot.urdf (robot description, URDF)
Before this commit: robot onshape, 2 links, 1 joints
Links:
- link part_1: geometry collision mesh filename=file:///TumDWM1001/Nav2Stuff/robocad/tum_block/part_1.stl; visual mesh filename=file:///TumDWM1001/Nav2Stuff/robocad/tum_block/part_1.stl
